File: probe-pcb/probe-pcb.kicad_sch (KiCad schematic)
At the start: 36 parts, among them J1 IDC_HEADER_02x08, J2 IDC_HEADER_2x12, U1 MIC5205-3.3YM5, U1 SN74AXC8T245, U2 DS90LV047A, U4 DS90LV047A

Commit message: Add 3d model for 2x12 pin header (missing in kicad library), add readme
Parts:
- J2: footprint Connector_IDC:IDC-Header_2x12_P2.54mm_Vertical -> idc:IDC-Header_2x12_P2.54mm_Vertical
Changed lines of the file:
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@@
       (effects (font (size 1.27 1.27)))
     )
-    (property "Footprint" "Connector_IDC:IDC-Header_2x12_P2.54mm_Vertical" (at 195.58 48.26 0)
+    (property "Footprint" "idc:IDC-Header_2x12_P2.54mm_Vertical" (at 195.58 48.26 0)
       (effects (font (size 1.27 1.27)) hide)
     )

Commit message: Change zener diodes to 3.9V (should protect both 3.3V and 5V level shifters)
Parts:
- D1: value 3.6V 2% -> 3.9V 5%; LCSC# C116949 -> C5359777; MPN MM3Z3V6T1G -> MM3Z3V9; Manufacturer onsemi -> Fosan
Other:
- note added: "Alternative part number for U1: SN74LXC8T245"
Changed lines of the file:
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@@
     (stroke (width 0) (type default))
+  )
+  (text "Alternative part number for U1: SN74LXC8T245" (at 29.21 105.41 0)
+    (effects (font (size 1.27 1.27)) (justify left bottom))
   )
   (label "D3_P" (at 140.97 113.03 0) (fields_autoplaced)
@@
       (effects (font (size 1.27 1.27)) (justify right))
     )
-    (property "Value" "3.6V 2%" (at 41.91 38.735 90)
+    (property "Value" "3.9V 5%" (at 41.91 38.735 90)
       (effects (font (size 1.27 1.27)) (justify right))
     )
@@
       (effects (font (size 1.27 1.27)) hide)
     )
-    (property "LCSC#" "C116949" (at 44.45 36.83 0)
-      (effects (font (size 1.27 1.27)) hide)
-    )
-    (property "MPN" "MM3Z3V6T1G" (at 44.45 36.83 0)
-      (effects (font (size 1.27 1.27)) hide)
-    )
-    (property "Manufacturer" "onsemi" (at 44.45 36.83 0)
-      (effects (font (size 1.27 1.27)) hide)
-    )
+    (property "LCSC#" "C5359777" (at 44.45 36.83 0)
+      (effects (font (size 1.27 1.27)) hide)
+    )
+    (property "MPN" "MM3Z3V9" (at 44.45 36.83 0)
+      (effects (font (size 1.27 1.27)) hide)
+    )
+    (property "Manufacturer" "Fosan" (at 44.45 36.83 0)
+      (effects (font (size 1.27 1.27)) hide)
+    )
