File: connector-pcb/connector-pcb.kicad_sch (KiCad schematic)
At the start: 39 parts, among them J1 MSO5000_LA, J2 IDC_HEADER_2x12, J3 IDC_HEADER_2x12, U1 MCP6002-xMS, U2 MCP6002-xMS

Commit message: Change connector PCB to 4 layer board, finalize probe board
Connections:
- net D0_N: now also J2.22 (Pin_22), R18.1; no longer J2.4 (Pin_4), R11.1
- net D0_P: now also J2.21 (Pin_21), R18.2; no longer J2.3 (Pin_3), R11.2
- net D10_N: now also J3.18 (Pin_18), R24.1; no longer J3.8 (Pin_8), R21.1
- net D10_P: now also J3.17 (Pin_17), R24.2; no longer J3.7 (Pin_7), R21.2
- net D11_N: now also J3.16 (Pin_16), R23.1; no longer J3.10 (Pin_10), R22.1
- net D11_P: now also J3.15 (Pin_15), R23.2; no longer J3.9 (Pin_9), R22.2
- net D12_N: now also J3.10 (Pin_10), R22.1; no longer J3.16 (Pin_16), R23.1
- net D12_P: now also J3.9 (Pin_9), R22.2; no longer J3.15 (Pin_15), R23.2
- net D13_N: now also J3.8 (Pin_8), R21.1; no longer J3.18 (Pin_18), R24.1
- net D13_P: now also J3.7 (Pin_7), R21.2; no longer J3.17 (Pin_17), R24.2
- net D14_N: now also J3.6 (Pin_6), R20.1; no longer J3.20 (Pin_20), R25.1
- net D14_P: now also J3.5 (Pin_5), R20.2; no longer J3.19 (Pin_19), R25.2
- net D15_N: now also J3.4 (Pin_4), R19.1; no longer J3.22 (Pin_22), R26.1
- net D15_P: now also J3.3 (Pin_3), R19.2; no longer J3.21 (Pin_21), R26.2
- net D1_N: now also J2.20 (Pin_20), R17.1; no longer J2.6 (Pin_6), R12.1
- net D1_P: now also J2.19 (Pin_19), R17.2; no longer J2.5 (Pin_5), R12.2
- net D2_N: now also J2.18 (Pin_18), R16.1; no longer J2.8 (Pin_8), R13.1
- net D2_P: now also J2.17 (Pin_17), R16.2; no longer J2.7 (Pin_7), R13.2
- net D3_N: now also J2.16 (Pin_16), R15.1; no longer J2.10 (Pin_10), R14.1
- net D3_P: now also J2.15 (Pin_15), R15.2; no longer J2.9 (Pin_9), R14.2
- net D4_N: now also J2.10 (Pin_10), R14.1; no longer J2.16 (Pin_16), R15.1
- net D4_P: now also J2.9 (Pin_9), R14.2; no longer J2.15 (Pin_15), R15.2
- net D5_N: now also J2.8 (Pin_8), R13.1; no longer J2.18 (Pin_18), R16.1
- net D5_P: now also J2.7 (Pin_7), R13.2; no longer J2.17 (Pin_17), R16.2
- net D6_N: now also J2.6 (Pin_6), R12.1; no longer J2.20 (Pin_20), R17.1
- net D6_P: now also J2.5 (Pin_5), R12.2; no longer J2.19 (Pin_19), R17.2
- net D7_N: now also J2.4 (Pin_4), R11.1; no longer J2.22 (Pin_22), R18.1
- net D7_P: now also J2.3 (Pin_3), R11.2; no longer J2.21 (Pin_21), R18.2
- net D8_N: now also J3.22 (Pin_22), R26.1; no longer J3.4 (Pin_4), R19.1
- net D8_P: now also J3.21 (Pin_21), R26.2; no longer J3.3 (Pin_3), R19.2
- net D9_N: now also J3.20 (Pin_20), R25.1; no longer J3.6 (Pin_6), R20.1
- net D9_P: now also J3.19 (Pin_19), R25.2; no longer J3.5 (Pin_5), R20.2

Commit message: Add 3d model for 2x12 pin header (missing in kicad library), add readme
Parts:
- J2, J3: footprint Connector_IDC:IDC-Header_2x12_P2.54mm_Vertical -> idc:IDC-Header_2x12_P2.54mm_Vertical
Changed lines of the file:
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@@
       (effects (font (size 1.27 1.27)))
     )
-    (property "Footprint" "Connector_IDC:IDC-Header_2x12_P2.54mm_Vertical" (at 157.48 88.9 0)
+    (property "Footprint" "idc:IDC-Header_2x12_P2.54mm_Vertical" (at 157.48 88.9 0)
       (effects (font (size 1.27 1.27)) hide)
     )
@@
       (effects (font (size 1.27 1.27)))
     )
-    (property "Footprint" "Connector_IDC:IDC-Header_2x12_P2.54mm_Vertical" (at 222.25 88.9 0)
-      (effects (font (size 1.27 1.27)) hide)
-    )
+    (property "Footprint" "idc:IDC-Header_2x12_P2.54mm_Vertical" (at 222.25 88.9 0)
+      (effects (font (size 1.27 1.27)) hide)
+    )

Commit message: Change zener diodes to 3.9V (should protect both 3.3V and 5V level shifters)
Parts:
- D1, D2: value 3.3V 2% -> 3.9V 5%; LCSC# C116949 -> C5359777; MPN MM3Z3V6T1G -> MM3Z3V9; Manufacturer onsemi -> Fosan
Changed lines of the file:
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@@
       (effects (font (size 1.27 1.27)) (justify left))
     )
-    (property "Value" "3.3V 2%" (at 76.2 32.385 90)
+    (property "Value" "3.9V 5%" (at 76.2 32.385 90)
       (effects (font (size 1.27 1.27)) (justify left))
     )
@@
       (effects (font (size 1.27 1.27)) hide)
     )
-    (property "LCSC#" "C116949" (at 73.66 30.48 0)
-      (effects (font (size 1.27 1.27)) hide)
-    )
-    (property "MPN" "MM3Z3V6T1G" (at 73.66 30.48 0)
-      (effects (font (size 1.27 1.27)) hide)
-    )
-    (property "Manufacturer" "onsemi" (at 73.66 30.48 0)
+    (property "LCSC#" "C5359777" (at 73.66 30.48 0)
+      (effects (font (size 1.27 1.27)) hide)
+    )
+    (property "MPN" "MM3Z3V9" (at 73.66 30.48 0)
+      (effects (font (size 1.27 1.27)) hide)
+    )
+    (property "Manufacturer" "Fosan" (at 73.66 30.48 0)
       (effects (font (size 1.27 1.27)) hide)
     )
@@
       (effects (font (size 1.27 1.27)) (justify left))
     )
-    (property "Value" "3.3V 2%" (at 204.47 33.655 90)
+    (property "Value" "3.9V 5%" (at 204.47 33.655 90)
       (effects (font (size 1.27 1.27)) (justify left))
     )
@@
       (effects (font (size 1.27 1.27)) hide)
     )
-    (property "LCSC#" "C116949" (at 201.93 31.75 0)
-      (effects (font (size 1.27 1.27)) hide)
-    )
-    (property "MPN" "MM3Z3V6T1G" (at 201.93 31.75 0)
-      (effects (font (size 1.27 1.27)) hide)
-    )
-    (property "Manufacturer" "onsemi" (at 201.93 31.75 0)
-      (effects (font (size 1.27 1.27)) hide)
-    )
+    (property "LCSC#" "C5359777" (at 201.93 31.75 0)
+      (effects (font (size 1.27 1.27)) hide)
+    )
+    (property "MPN" "MM3Z3V9" (at 201.93 31.75 0)
+      (effects (font (size 1.27 1.27)) hide)
+    )
+    (property "Manufacturer" "Fosan" (at 201.93 31.75 0)
+      (effects (font (size 1.27 1.27)) hide)
+    )

Commit message: Changed R9 of connector PCB from 10k to 100R (otherwise the scope wouldn't detect the probes)
Parts:
- R9: value 10K -> 100R; LCSC# C98220 -> C105588; MPN RC0603FR-0710KL -> RC0603FR-07100RL
Changed lines of the file:
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@@
       (effects (font (size 1.27 1.27)))
     )
-    (property "Value" "10K" (at 40.64 74.93 90)
+    (property "Value" "100R" (at 40.64 74.93 90)
       (effects (font (size 1.27 1.27)))
     )
@@
       (effects (font (size 1.27 1.27)) hide)
     )
-    (property "LCSC#" "C98220" (at 40.64 77.47 0)
+    (property "LCSC#" "C105588" (at 40.64 77.47 0)
       (effects (font (size 1.27 1.27)) hide)
     )
-    (property "MPN" "RC0603FR-0710KL" (at 40.64 77.47 0)
+    (property "MPN" "RC0603FR-07100RL" (at 40.64 77.47 0)
       (effects (font (size 1.27 1.27)) hide)
     )
